File: PCBs/DC-DC Board/DC-DC Board.sch (KiCad schematic (older format))
At the start: 37 parts, among them J1 Conn_01x01, J2 Conn_01x01, J3 Conn_01x01, J4 Conn_01x01, J5 Conn_01x02, J6 Conn_01x02, Q1 Q_NMOS_DGS, U1 MurataDC-DC, U2 ACS711, U3 NCP551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

Commit message: DC-DC Board DONE
Should be done for sure now bys
Parts:
- removed D2: LED, LEDs:LED_0805, symbol Device:LED
- removed Q1: Q_NMOS_DGS, EER:SOT-23-NMOS, symbol Device:Q_NMOS_DGS
- removed R5: 1k, Resistors_SMD:R_0805, symbol Device:R
- added Q1: Q_NMOS_GDS, TO_SOT_Packages_SMD:TO-252-2, symbol Device:Q_NMOS_GDS
- added R9: 0, Resistors_SMD:R_0603, symbol Device:R
- R7: value 100k -> 200k
Connections:
- net labels removed: GND_Surface, PG, SMBALERT
- wire segments 156 -> 149
- no-connect marks 0 -> 2
Other:
- note added: "Reverse Voltage\nPolarity Protection\n"
- note removed: "LED lights if fault detected"
- note removed: "Reverse Polarity\nVoltage Protection\n"
Changed lines of the file:
@@
 L Connector_Generic:Conn_01x01 J1
 U 1 1 5BBFE9D3
-P 1855 4390
-F 0 "J1" H 1775 4165 50  0000 C CNN
-F 1 "Conn_01x01" H 1775 4256 50  0000 C CNN
-F 2 "EER:RingTerminal" H 1855 4390 50  0001 C CNN
-F 3 "~" H 1855 4390 50  0001 C CNN
-	1    1855 4390
+P 1490 4390
+F 0 "J1" H 1410 4165 50  0000 C CNN
+F 1 "Conn_01x01" H 1410 4256 50  0000 C CNN
+F 2 "EER:RingTerminal" H 1490 4390 50  0001 C CNN
+F 3 "~" H 1490 4390 50  0001 C CNN
+	1    1490 4390
 	-1   0    0    1
 $EndComp
@@
 Text Label 1850 1690 0    50   ~ 0
 +48V
-Text Label 2135 4390 0    50   ~ 0
-GND_Surface
 $Comp
 L Connector_Generic:Conn_01x01 J4
@@
 $EndComp
 Wire Wire Line
-	6550 2090 6550 2290
-Text GLabel 6400 2290 0    50   Input ~ 0
-PG
-Wire Wire Line
-	6400 2290 6550 2290
-$Comp
-L Device:R R5
-U 1 1 5BC29904
-P 6550 1940
-F 0 "R5" H 6620 1986 50  0000 L CNN
-F 1 "1k" H 6620 1895 50  0000 L CNN
-F 2 "Resistors_SMD:R_0805" V 6480 1940 50  0001 C CNN
-F 3 "~" H 6550 1940 50  0001 C CNN
-	1    6550 1940
-	1    0    0    -1
-$EndComp
-$Comp
-L Device:LED D2
-U 1 1 5BC29944
-P 6550 1490
-F 0 "D2" V 6588 1373 50  0000 R CNN
-F 1 "LED" V 6497 1373 50  0000 R CNN
-F 2 "LEDs:LED_0805" H 6550 1490 50  0001 C CNN
-F 3 "~" H 6550 1490 50  0001 C CNN
-	1    6550 1490
-	0    -1   -1   0
-$EndComp
-Wire Wire Line
-	6550 1790 6550 1640
-Wire Wire Line
 	6950 2090 6950 2340
 $Comp
@@
 	1    0    0    -1
 $EndComp
-Wire Wire Line
-	6950 1190 6950 1340
 $Comp
 L power:+12V #PWR0106
 U 1 1 5BC2C731
-P 6750 1040
-F 0 "#PWR0106" H 6750 890 50  0001 C CNN
-F 1 "+12V" H 6765 1213 50  0000 C CNN
-F 2 "" H 6750 1040 50  0001 C CNN
-F 3 "" H 6750 1040 50  0001 C CNN
-	1    6750 1040
-	1    0    0    -1
-$EndComp
-Wire Wire Line
-	6750 1040 6750 1190
-Wire Wire Line
-	6750 1190 6950 1190
-Wire Wire Line
-	6550 1340 6550 1190
-Wire Wire Line
-	6550 1190 6750 1190
-Connection ~ 6750 1190
+P 6950 1040
+F 0 "#PWR0106" H 6950 890 50  0001 C CNN
+F 1 "+12V" H 6965 1213 50  0000 C CNN
+F 2 "" H 6950 1040 50  0001 C CNN
+F 3 "" H 6950 1040 50  0001 C CNN
+	1    6950 1040
+	1    0    0    -1
+$EndComp
 $Comp
 L Connector_Generic:Conn_01x02 J5
@@
 Text GLabel 4390 1790 2    50   Input ~ 0
 VIOUT
-Text GLabel 6050 3440 2    50   Input ~ 0
-SMBALERT
-Text GLabel 6050 3640 2    50   Input ~ 0
-PG
 Text GLabel 6050 3740 2    50   Input ~ 0
 SDA
 Text GLabel 6050 3840 2    50   Input ~ 0
 SCL
-Wire Wire Line
-	6050 3640 5800 3640
 Wire Wire Line
 	6050 3740 5800 3740
@@
 Text Notes 765  2965 0    50   ~ 0
 1/4 W MINIMUM\n
-Text Notes 5800 1990 0    50   ~ 0
+Text Notes 6190 1970 0    50   ~ 0
 1/8 W MINIMUM\n
 $Comp
@@
 Text Notes 8100 3090 0    50   ~ 0
 Output Filtering
-Text Notes 5400 1540 0    50   ~ 0
-LED lights if fault detected
 Text Notes 8900 1240 0    50   ~ 0
 SMBUS\n
@@
 Text Notes 9100 4240 0    50   ~ 0
 ROV Ground\n
-Text Notes 3450 4690 0    50   ~ 0
+Text Notes 1270 4580 0    50   ~ 0
 Surface Ground
 $Bitmap
@@
 Wire Wire Line
 	6150 4620 6150 4390
-Wire Wire Line
-	5800 3440 6050 3440
 $Comp
 L Device:C C12
@@
 Text Notes 1500 1045 0    39   Italic 0
 Because of layout considerations, this current sensor is wired "backwards"\nfrom what it normally should be. This just means we are reading a negative \ncurrent when it should be positive. Simple software fix.\n
-Text Notes 3230 3605 0    50   Italic 10
-Reverse Polarity\nVoltage Protection\n
+Text Notes 1950 3960 0    50   Italic 10
+Reverse Voltage\nPolarity Protection\n
 $Comp
 L Device:R R1
@@
 P 2960 3990
 F 0 "R7" H 3030 4036 50  0000 L CNN
-F 1 "100k" H 3030 3945 50  0000 L CNN
+F 1 "200k" H 3030 3945 50  0000 L CNN
 F 2 "Resistors_SMD:R_0603" V 2890 3990 50  0001 C CNN
 F 3 "~" H 2960 3990 50  0001 C CNN
@@
 $EndComp
 Wire Wire Line
-	2960 3720 2960 3780
-Wire Wire Line
 	1840 3190 2960 3190
 Wire Wire Line
-	2055 4390 2960 4390
-Wire Wire Line
-	3300 4085 3250 4085
-Wire Wire Line
-	3250 4085 3250 3780
-Wire Wire Line
-	3250 3780 2960 3780
-Connection ~ 2960 3780
-Wire Wire Line
-	2960 3780 2960 3840
-Wire Wire Line
-	3600 3885 3600 3790
-Wire Wire Line
 	3300 4390 3600 4390
-$Comp
-L Device:Q_NMOS_DGS Q1
-U 1 1 5BCCC58A
-P 3500 4085
-F 0 "Q1" H 3705 4131 50  0000 L CNN
-F 1 "Q_NMOS_DGS" H 3080 3910 50  0000 L CNN
-F 2 "EER:SOT-23-NMOS" H 3700 4185 50  0001 C CNN
-F 3 "~" H 3500 4085 50  0001 C CNN
-	1    3500 4085
-	1    0    0    -1
-$EndComp
-Wire Wire Line
-	3600 4285 3600 4390
 Connection ~ 3600 4390
 Wire Wire Line
@@
 Wire Wire Line
 	2960 4140 2960 4390
+Wire Wire Line
+	2960 4390 3300 4390
+NoConn ~ 5800 3440
+NoConn ~ 5800 3640
+$Comp
+L Device:R R9
+U 1 1 5BD454F0
+P 3600 4080
+F 0 "R9" H 3670 4126 50  0000 L CNN
+F 1 "0" H 3670 4035 50  0000 L CNN
+F 2 "Resistors_SMD:R_0603" V 3530 4080 50  0001 C CNN
+F 3 "~" H 3600 4080 50  0001 C CNN
+	1    3600 4080
+	1    0    0    -1
+$EndComp
+Wire Wire Line
+	3600 3790 3600 3930
+Wire Wire Line
+	3600 4230 3600 4390
+Wire Wire Line
+	2960 3720 2960 3780
+$Comp
+L Device:Q_NMOS_GDS Q1
+U 1 1 5BD739CF
+P 2340 4490
+F 0 "Q1" V 2683 4490 50  0000 C CNN
+F 1 "Q_NMOS_GDS" V 2592 4490 50  0000 C CNN
+F 2 "TO_SOT_Packages_SMD:TO-252-2" H 2540 4590 50  0001 C CNN
+F 3 "~" H 2340 4490 50  0001 C CNN
+	1    2340 4490
+	0    -1   -1   0
+$EndComp
+Wire Wire Line
+	2540 4390 2960 4390
+Wire Wire Line
+	2960 4390 2960 4380
 Connection ~ 2960 4390
 Wire Wire Line
-	2960 4390 3300 4390
+	2140 4390 1690 4390
+Wire Wire Line
+	2340 4690 2740 4690
+Wire Wire Line
+	2740 4690 2740 3780
+Wire Wire Line
+	2740 3780 2960 3780
+Connection ~ 2960 3780
+Wire Wire Line
+	2960 3780 2960 3840
+Wire Wire Line
+	6950 1040 6950 1340
 $EndSCHEMATC

Commit message: Cleaned up BOM
KiCAD has a built in BOM!! Woohooo!!!
Parts:
- R1: value 700k -> 698k
- U1: value MurataDC-DC -> DBQ0135V2
Changed lines of the file:
@@
 P 4850 3790
 F 0 "U1" H 4850 4655 50  0000 C CNN
-F 1 "MurataDC-DC" H 4850 4564 50  0000 C CNN
+F 1 "DBQ0135V2" H 4850 4564 50  0000 C CNN
 F 2 "EER:MurataDC-DC" H 4850 3790 50  0001 C CNN
-F 3 "" H 4850 3790 50  0001 C CNN
+F 3 "S5801-05-ND" H 4850 3790 50  0001 C CNN
 	1    4850 3790
 	1    0    0    -1
@@
 F 1 "Conn_01x01" H 1410 4256 50  0000 C CNN
 F 2 "EER:RingTerminal" H 1490 4390 50  0001 C CNN
-F 3 "~" H 1490 4390 50  0001 C CNN
+F 3 "36-7770-ND" H 1490 4390 50  0001 C CNN
 	1    1490 4390
 	-1   0    0    1
@@
 F 1 "Conn_01x01" H 1275 1556 50  0000 C CNN
 F 2 "EER:RingTerminal" H 1355 1690 50  0001 C CNN
-F 3 "~" H 1355 1690 50  0001 C CNN
+F 3 "36-7770-ND" H 1355 1690 50  0001 C CNN
 	1    1355 1690
 	-1   0    0    1
@@
 F 1 "Conn_01x01" H 9230 3141 50  0000 L CNN
 F 2 "EER:RingTerminal" H 9150 3190 50  0001 C CNN
-F 3 "~" H 9150 3190 50  0001 C CNN
+F 3 "36-7770-ND" H 9150 3190 50  0001 C CNN
 	1    9150 3190
 	1    0    0    -1
@@
 F 1 "Conn_01x01" H 9230 4341 50  0000 L CNN
 F 2 "EER:RingTerminal" H 9150 4390 50  0001 C CNN
-F 3 "~" H 9150 4390 50  0001 C CNN
+F 3 "36-7770-ND" H 9150 4390 50  0001 C CNN
 	1    9150 4390
 	1    0    0    -1
@@
 F 1 "ACS711" H 2850 2364 50  0000 C CNN
 F 2 "EER:ACS711" H 2750 1940 50  0001 C CNN
-F 3 "" H 2750 1940 50  0001 C CNN
+F 3 "620-1482-1-ND" H 2750 1940 50  0001 C CNN
 	1    2850 1940
 	1    0    0    -1
@@
 F 1 "0" H 6920 4045 50  0001 L CNN
 F 2 "Resistors_SMD:R_0805" V 6780 4090 50  0001 C CNN
-F 3 "~" H 6850 4090 50  0001 C CNN
+F 3 "RNCP0805FTD10K0CT-ND" H 6850 4090 50  0001 C CNN
 	1    6850 4090
 	1    0    0    -1
@@
 F 1 "0" H 6220 4045 50  0001 L CNN
 F 2 "Resistors_SMD:R_0805" V 6080 4090 50  0001 C CNN
-F 3 "~" H 6150 4090 50  0001 C CNN
+F 3 "RMCF0805FT22K0CT-ND" H 6150 4090 50  0001 C CNN
 	1    6150 4090
 	1    0    0    -1
@@
 Wire Wire Line
 	5800 4040 6050 4040
-Wire Wire Line
-	6050 4040 6050 3890
-Wire Wire Line
-	6850 3890 6850 3940
 Wire Wire Line
 	6850 4240 6850 4390
@@
 F 1 "4.7nF" H 6565 4045 50  0000 L CNN
 F 2 "Capacitors_SMD:C_0805" H 6488 3940 50  0001 C CNN
-F 3 "~" H 6450 4090 50  0001 C CNN
+F 3 "399-9092-1-ND" H 6450 4090 50  0001 C CNN
 	1    6450 4090
 	1    0    0    -1
@@
 F 1 "4.7nF" H 7265 4045 50  0000 L CNN
 F 2 "Capacitors_SMD:C_0805" H 7188 3940 50  0001 C CNN
-F 3 "~" H 7150 4090 50  0001 C CNN
+F 3 "399-9092-1-ND" H 7150 4090 50  0001 C CNN
 	1    7150 4090
 	1    0    0    -1
@@
 Wire Wire Line
 	6150 4390 6450 4390
-Wire Wire Line
-	6850 3890 7150 3890
-Wire Wire Line
-	7150 3890 7150 3940
-Connection ~ 6850 3890
 Wire Wire Line
 	7150 4240 7150 4390
@@
 Wire Wire Line
 	6850 4390 7150 4390
-Wire Wire Line
-	6050 3890 6850 3890
 $Comp
 L Device:LED D3
@@
 F 1 "LED" V 6897 1373 50  0000 R CNN
 F 2 "LEDs:LED_0805" H 6950 1490 50  0001 C CNN
-F 3 "~" H 6950 1490 50  0001 C CNN
+F 3 "732-4982-1-ND" H 6950 1490 50  0001 C CNN
 	1    6950 1490
 	0    -1   -1   0
@@
 F 1 "1k" H 7020 1895 50  0000 L CNN
 F 2 "Resistors_SMD:R_0805" V 6880 1940 50  0001 C CNN
-F 3 "~" H 6950 1940 50  0001 C CNN
+F 3 "RNCP0805FTD1K00CT-ND" H 6950 1940 50  0001 C CNN
 	1    6950 1940
 	1    0    0    -1
@@
 F 1 "Conn_01x02" H 9130 1291 50  0000 L CNN
 F 2 "EER:MOLEX_0705530001" H 9050 1390 50  0001 C CNN
-F 3 "~" H 9050 1390 50  0001 C CNN
+F 3 "WM4900-ND" H 9050 1390 50  0001 C CNN
 	1    9050 1390
 	1    0    0    -1
@@
 F 1 "Conn_01x02" H 9130 1791 50  0000 L CNN
 F 2 "EER:MOLEX_0705530001" H 9050 1890 50  0001 C CNN
-F 3 "~" H 9050 1890 50  0001 C CNN
+F 3 "WM4900-ND" H 9050 1890 50  0001 C CNN
 	1    9050 1890
 	1    0    0    -1
@@
 F 1 "47uF" H 8065 3695 50  0000 L CNN
 F 2 "Capacitors_THT:CP_Radial_D6.3mm_P2.50mm" H 7950 3740 50  0001 C CNN
-F 3 "~" H 7950 3740 50  0001 C CNN
+F 3 "399-13665-ND" H 7950 3740 50  0001 C CNN
 	1    7950 3740
 	1    0    0    -1
@@
 F 1 "220uF" H 8515 3695 50  0000 L CNN
 F 2 "Capacitors_THT:CP_Radial_D6.3mm_P2.50mm" H 8400 3740 50  0001 C CNN
-F 3 "~" H 8400 3740 50  0001 C CNN
+F 3 "399-13664-ND" H 8400 3740 50  0001 C CNN
 	1    8400 3740
 	1    0    0    -1
@@
 F 1 "220uF" H 8965 3695 50  0000 L CNN
 F 2 "Capacitors_THT:CP_Radial_D6.3mm_P2.50mm" H 8850 3740 50  0001 C CNN
-F 3 "~" H 8850 3740 50  0001 C CNN
+F 3 "399-13664-ND" H 8850 3740 50  0001 C CNN
 	1    8850 3740
 	1    0    0    -1
@@
 F 1 "1uF" H 7255 5415 50  0000 L CNN
 F 2 "Capacitors_SMD:C_0805" H 7178 5310 50  0001 C CNN
-F 3 "~" H 7140 5460 50  0001 C CNN
+F 3 "399-1284-1-ND" H 7140 5460 50  0001 C CNN
 	1    7140 5460
 	1    0    0    -1
@@
 F 1 "1uF" H 8255 5415 50  0000 L CNN
 F 2 "Capacitors_SMD:C_0805" H 8178 5310 50  0001 C CNN
-F 3 "~" H 8140 5460 50  0001 C CNN
+F 3 "399-1284-1-ND" H 8140 5460 50  0001 C CNN
 	1    8140 5460
 	1    0    0    -1
@@
 F 1 "1uF" H 8755 5415 50  0000 L CNN
 F 2 "Capacitors_SMD:C_0805" H 8678 5310 50  0001 C CNN
-F 3 "~" H 8640 5460 50  0001 C CNN
+F 3 "399-1284-1-ND" H 8640 5460 50  0001 C CNN
 	1    8640 5460
 	1    0    0    -1
@@
 F 1 "1uF" H 9755 5415 50  0000 L CNN
 F 2 "Capacitors_SMD:C_0805" H 9678 5310 50  0001 C CNN
-F 3 "~" H 9640 5460 50  0001 C CNN
+F 3 "399-1284-1-ND" H 9640 5460 50  0001 C CNN
 	1    9640 5460
 	1    0    0    -1
@@
 F 1 "0.1uF" H 4265 1950 50  0000 L CNN
 F 2 "Capacitors_SMD:C_0805" H 4188 1845 50  0001 C CNN
-F 3 "~" H 4150 1995 50  0001 C CNN
+F 3 "399-1169-1-ND" H 4150 1995 50  0001 C CNN
 	1    4150 1995
 	1    0    0    -1
@@
 F 1 "LED" V 1412 2398 50  0000 R CNN
 F 2 "LEDs:LED_0805" H 1465 2515 50  0001 C CNN
-F 3 "~" H 1465 2515 50  0001 C CNN
+F 3 "732-4983-1-ND" H 1465 2515 50  0001 C CNN
 	1    1465 2515
 	0    -1   -1   0
@@
 F 1 "10k" H 1535 2920 50  0000 L CNN
 F 2 "Resistors_SMD:R_0805" V 1395 2965 50  0001 C CNN
-F 3 "~" H 1465 2965 50  0001 C CNN
+F 3 "RNCP0805FTD10K0CT-ND" H 1465 2965 50  0001 C CNN
 	1    1465 2965
 	1    0    0    -1
@@
 F 1 "1k" H 3590 1930 50  0000 L CNN
 F 2 "Resistors_SMD:R_0805" V 3450 1975 50  0001 C CNN
-F 3 "~" H 3520 1975 50  0001 C CNN
+F 3 "RNCP0805FTD1K00CT-ND" H 3520 1975 50  0001 C CNN
 	1    3520 1975
 	1    0    0    -1
@@
 F 1 "1uF" H 3905 1950 50  0000 L CNN
 F 2 "Capacitors_SMD:C_0805" H 3828 1845 50  0001 C CNN
-F 3 "~" H 3790 1995 50  0001 C CNN
+F 3 "399-1284-1-ND" H 3790 1995 50  0001 C CNN
 	1    3790 1995
 	1    0    0    -1
@@
 F 1 "1uF" H 10135 5415 50  0000 L CNN
 F 2 "Capacitors_SMD:C_0805" H 10058 5310 50  0001 C CNN
-F 3 "~" H 10020 5460 50  0001 C CNN
+F 3 "399-1284-1-ND" H 10020 5460 50  0001 C CNN
 	1    10020 5460
 	1    0    0    -1
@@
 F 1 "0.1uF" H 10505 5415 50  0000 L CNN
 F 2 "Capacitors_SMD:C_0805" H 10428 5310 50  0001 C CNN
-F 3 "~" H 10390 5460 50  0001 C CNN
+F 3 "399-1169-1-ND" H 10390 5460 50  0001 C CNN
 	1    10390 5460
 	1    0    0    -1
@@
 P 2960 3570
 F 0 "R1" H 3030 3616 50  0000 L CNN
-F 1 "700k" H 3030 3525 50  0000 L CNN
+F 1 "698k" H 3030 3525 50  0000 L CNN
 F 2 "Resistors_SMD:R_0603" V 2890 3570 50  0001 C CNN
-F 3 "~" H 2960 3570 50  0001 C CNN
+F 3 "RMCF0603FT698KCT-ND" H 2960 3570 50  0001 C CNN
 	1    2960 3570
 	1    0    0    -1
@@
 F 1 "200k" H 3030 3945 50  0000 L CNN
 F 2 "Resistors_SMD:R_0603" V 2890 3990 50  0001 C CNN
-F 3 "~" H 2960 3990 50  0001 C CNN
+F 3 "RMCF0603JT200KCT-ND" H 2960 3990 50  0001 C CNN
 	1    2960 3990
 	1    0    0    -1
@@
 F 1 "0" H 3670 4035 50  0000 L CNN
 F 2 "Resistors_SMD:R_0603" V 3530 4080 50  0001 C CNN
-F 3 "~" H 3600 4080 50  0001 C CNN
+F 3 "RMCF0603ZT0R00CT-ND" H 3600 4080 50  0001 C CNN
 	1    3600 4080
 	1    0    0    -1
@@
 F 1 "Q_NMOS_GDS" V 2592 4490 50  0000 C CNN
 F 2 "TO_SOT_Packages_SMD:TO-252-2" H 2540 4590 50  0001 C CNN
-F 3 "~" H 2340 4490 50  0001 C CNN
+F 3 "DMTH6004SK3-13DICT-ND" H 2340 4490 50  0001 C CNN
 	1    2340 4490
 	0    -1   -1   0
@@
 Wire Wire Line
 	6950 1040 6950 1340
+Wire Wire Line
+	6850 3910 6850 3940
+Wire Wire Line
+	7150 3910 7150 3940
+Wire Wire Line
+	7150 3910 6850 3910
+Wire Wire Line
+	6850 3910 6050 3910
+Wire Wire Line
+	6050 3910 6050 4040
+Connection ~ 6850 3910
 $EndSCHEMATC
