File: PCBs/DC-DC Board/_saved_DC-DC Board.sch (KiCad schematic (older format))
At the start: 37 parts, among them J1 Conn_01x01, J2 Conn_01x01, J3 Conn_01x01, J4 Conn_01x01, J5 Conn_01x02, J6 Conn_01x02, Q1 Q_NMOS_DGS, U1 MurataDC-DC, U2 ACS711, U3 NCP551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

Commit message: Added Reverse Polarity Protection
Accomplished with an NMOS on the primary on/off pin. Still need to verify this is OK in the lab.
Other:
- note added: "Reverse Voltage\nPolarity Protection\n"
- note removed: "Reverse Polarity\nVoltage Protection\n"
Changed lines of the file:
@@
 Because of layout considerations, this current sensor is wired "backwards"\nfrom what it normally should be. This just means we are reading a negative \ncurrent when it should be positive. Simple software fix.\n
 Text Notes 3230 3605 0    50   Italic 10
-Reverse Polarity\nVoltage Protection\n
+Reverse Voltage\nPolarity Protection\n
 $Comp
 L Device:R R1
