File: PCBs/Dual CamCon/Dual CamCon.sch (KiCad schematic (older format))
At the start: 7 parts, among them J1 Servo Input, J2 Servo Input, J3 Camera FPC Connector, J4 Camera FPC Connector, J5 Raspberry Pi GPIO, P1 HDMI Connector, P2 HDMI Connector

Commit message: Finished Mechanicals of the Dual CamCon Board
Just need to do the routing now.
Parts:
- added C1, C2, C3, C4: C, EER:C_0805_HandSoldering, symbol Device:C
Connections:
- net labels added: CAM1_3V3, CAM1_CLK, CAM1_CN, CAM1_CP, CAM1_DN0, CAM1_DN1, CAM1_DP0, CAM1_DP1, CAM1_GPIO, CAM1_SCL, CAM1_SDA, CAM2_3V3, CAM2_CLK, CAM2_CN, CAM2_CP, CAM2_DN0, CAM2_DN1, CAM2_DP0, CAM2_DP1, CAM2_GPIO, CAM2_SCL, CAM2_SDA, Servo1, Servo2
- wire segments 22 -> 136
- no-connect marks 0 -> 30
Other:
- note added: "Eastern Edge Robotics"
- note added: "Filtering caps incase the servo signal is jittery\n"
- note added: "If need be, we can solder to \nthe top Pi's GPIOs as a last ditch fix for something\n"
- note added: "Mark Belbin\n"
- note added: "Oct. 2018"
- note added: "Powering the servos with the Pis +5V"
- note added: "Trying to match sensitive signals\nwith shielded twisted pairs"

Commit message: Dual CamCon Board - Ready for Review
Pretty much cleaned up this guy as much as I could. Needs to be reviewed by the team on a few different things.

-FPC to HDMI legitness (will each pin line up) needs to be triple checked.
Connections:
- net labels added: CAM1_C+, CAM1_C-, CAM1_D0+, CAM1_D0-, CAM1_D1+, CAM1_D1-, CAM2_C+, CAM2_C-, CAM2_D0+, CAM2_D0-, CAM2_D1+, CAM2_D1-
- net labels removed: CAM1_CN, CAM1_CP, CAM1_DN0, CAM1_DN1, CAM1_DP0, CAM1_DP1, CAM2_CN, CAM2_CP, CAM2_DN0, CAM2_DN1, CAM2_DP0, CAM2_DP1
Changed lines of the file:
@@
 EESchema Schematic File Version 4
+LIBS:Dual CamCon-cache
 EELAYER 26 0
 EELAYER END
@@
 	3250 5700 3250 6300
 Text Label 3350 2750 0    50   ~ 0
-CAM1_DN0
+CAM1_D0-
 Text Label 3350 2850 0    50   ~ 0
-CAM1_DP0
+CAM1_D0+
 Text Label 3350 3050 0    50   ~ 0
-CAM1_DN1
+CAM1_D1-
 Text Label 3350 3150 0    50   ~ 0
-CAM1_DP1
+CAM1_D1+
 Text Label 3350 3350 0    50   ~ 0
-CAM1_CN
+CAM1_C-
 Text Label 3350 3450 0    50   ~ 0
-CAM1_CP
+CAM1_C+
 Text Label 3350 3650 0    50   ~ 0
 CAM1_GPIO
@@
 	3350 4050 3750 4050
 Text Label 3350 4900 0    50   ~ 0
-CAM2_DN0
+CAM2_D0-
 Text Label 3350 5000 0    50   ~ 0
-CAM2_DP0
+CAM2_D0+
 Text Label 3350 5200 0    50   ~ 0
-CAM2_DN1
+CAM2_D1-
 Text Label 3350 5300 0    50   ~ 0
-CAM2_DP1
+CAM2_D1+
 Text Label 3350 5500 0    50   ~ 0
-CAM2_CN
+CAM2_C-
 Text Label 3350 5600 0    50   ~ 0
-CAM2_CP
+CAM2_C+
 Text Label 3350 5800 0    50   ~ 0
 CAM2_GPIO
@@
 	5850 2700 6000 2700
 Text Label 5850 4400 0    50   ~ 0
-CAM1_DN0
+CAM1_D0-
 Text Label 5850 4200 0    50   ~ 0
-CAM1_DP0
+CAM1_D0+
 Wire Wire Line
 	5850 4000 6350 4000
@@
 	5850 3500 6250 3500
 Text Label 5850 4100 0    50   ~ 0
-CAM1_DN1
+CAM1_D1-
 Text Label 5850 3900 0    50   ~ 0
-CAM1_DP1
+CAM1_D1+
 Text Label 5850 3800 0    50   ~ 0
-CAM1_CN
+CAM1_C-
 Text Label 5850 3600 0    50   ~ 0
-CAM1_CP
+CAM1_C+
 Text Label 5850 3500 0    50   ~ 0
 CAM1_GPIO
@@
 	5850 6550 6250 6550
 Text Label 5850 6550 0    50   ~ 0
-CAM2_DN0
+CAM2_D0-
 Text Label 5850 6350 0    50   ~ 0
-CAM2_DP0
+CAM2_D0+
 Text Label 5850 6250 0    50   ~ 0
-CAM2_DN1
+CAM2_D1-
 Text Label 5850 6050 0    50   ~ 0
-CAM2_DP1
+CAM2_D1+
 Text Label 5850 5950 0    50   ~ 0
-CAM2_CN
+CAM2_C-
 Text Label 5850 5750 0    50   ~ 0
-CAM2_CP
+CAM2_C+
 Text Label 5850 5650 0    50   ~ 0
 CAM2_GPIO

Commit message: Major Routing Fix for Dual CamCon
After looking at the physical Pi Cam I realized that I had the pin map mirrored. I swapped the pins around on the FPC connector and cleaned up the board in general. Count this as a double check, still need another check from someone else.
Other:
- note added: "Trying to match differential signals\nwith shielded twisted pairs"
- note removed: "Trying to match sensitive signals\nwith shielded twisted pairs"
Changed lines of the file:
@@
 $EndComp
-Wire Wire Line
-	3250 2650 3250 2950
-Wire Wire Line
-	3750 4150 3250 4150
-Connection ~ 3250 4150
-Wire Wire Line
-	3250 4150 3250 4250
-Wire Wire Line
-	3750 4250 3250 4250
-Connection ~ 3250 4250
-Wire Wire Line
-	3250 4250 3250 4800
 Wire Wire Line
 	3750 6400 3250 6400
@@
 Wire Wire Line
 	3250 6300 3250 6400
-Wire Wire Line
-	3750 2950 3250 2950
-Connection ~ 3250 2950
-Wire Wire Line
-	3250 2950 3250 3250
-Wire Wire Line
-	3750 3250 3250 3250
-Connection ~ 3250 3250
-Wire Wire Line
-	3250 3250 3250 3550
-Wire Wire Line
-	3750 3550 3250 3550
-Connection ~ 3250 3550
-Wire Wire Line
-	3250 3550 3250 4150
-Wire Wire Line
-	3750 2650 3250 2650
-Wire Wire Line
-	3750 4800 3250 4800
-Connection ~ 3250 4800
-Wire Wire Line
-	3250 4800 3250 5100
-Wire Wire Line
-	3750 5100 3250 5100
-Connection ~ 3250 5100
-Wire Wire Line
-	3250 5100 3250 5400
-Wire Wire Line
-	3750 5400 3250 5400
-Connection ~ 3250 5400
-Wire Wire Line
-	3250 5400 3250 5700
-Wire Wire Line
-	3750 5700 3250 5700
-Connection ~ 3250 5700
-Wire Wire Line
-	3250 5700 3250 6300
-Text Label 3350 2750 0    50   ~ 0
+Text Label 3350 3950 0    50   ~ 0
 CAM1_D0-
-Text Label 3350 2850 0    50   ~ 0
+Text Label 3350 3850 0    50   ~ 0
 CAM1_D0+
-Text Label 3350 3050 0    50   ~ 0
+Text Label 3350 3650 0    50   ~ 0
 CAM1_D1-
-Text Label 3350 3150 0    50   ~ 0
+Text Label 3350 3550 0    50   ~ 0
 CAM1_D1+
 Text Label 3350 3350 0    50   ~ 0
 CAM1_C-
-Text Label 3350 3450 0    50   ~ 0
+Text Label 3350 3250 0    50   ~ 0
 CAM1_C+
-Text Label 3350 3650 0    50   ~ 0
+Text Label 3350 3050 0    50   ~ 0
 CAM1_GPIO
-Text Label 3350 3750 0    50   ~ 0
+Text Label 3350 2950 0    50   ~ 0
 CAM1_CLK
-Text Label 3350 3850 0    50   ~ 0
+Text Label 3350 2850 0    50   ~ 0
 CAM1_SCL
-Text Label 3350 3950 0    50   ~ 0
+Text Label 3350 2750 0    50   ~ 0
 CAM1_SDA
-Text Label 3350 4050 0    50   ~ 0
+Text Label 3350 2650 0    50   ~ 0
 CAM1_3V3
 Wire Wire Line
@@
 	3350 2850 3750 2850
 Wire Wire Line
-	3350 3150 3750 3150
-Wire Wire Line
 	3350 3050 3750 3050
 Wire Wire Line
 	3350 3350 3750 3350
 Wire Wire Line
-	3350 3450 3750 3450
-Wire Wire Line
 	3350 3650 3750 3650
 Wire Wire Line
-	3350 3750 3750 3750
-Wire Wire Line
 	3350 3850 3750 3850
 Wire Wire Line
 	3350 3950 3750 3950
-Wire Wire Line
-	3350 4050 3750 4050
-Text Label 3350 4900 0    50   ~ 0
+Text Label 3350 6100 0    50   ~ 0
 CAM2_D0-
-Text Label 3350 5000 0    50   ~ 0
+Text Label 3350 6000 0    50   ~ 0
 CAM2_D0+
-Text Label 3350 5200 0    50   ~ 0
+Text Label 3350 5800 0    50   ~ 0
 CAM2_D1-
-Text Label 3350 5300 0    50   ~ 0
+Text Label 3350 5700 0    50   ~ 0
 CAM2_D1+
 Text Label 3350 5500 0    50   ~ 0
 CAM2_C-
-Text Label 3350 5600 0    50   ~ 0
+Text Label 3350 5400 0    50   ~ 0
 CAM2_C+
-Text Label 3350 5800 0    50   ~ 0
+Text Label 3350 5200 0    50   ~ 0
 CAM2_GPIO
-Text Label 3350 5900 0    50   ~ 0
+Text Label 3350 5100 0    50   ~ 0
 CAM2_CLK
-Text Label 3350 6000 0    50   ~ 0
+Text Label 3350 5000 0    50   ~ 0
 CAM2_SCL
-Text Label 3350 6100 0    50   ~ 0
+Text Label 3350 4900 0    50   ~ 0
 CAM2_SDA
-Text Label 3350 6200 0    50   ~ 0
+Text Label 3350 4800 0    50   ~ 0
 CAM2_3V3
 Wire Wire Line
@@
 	3350 5200 3750 5200
 Wire Wire Line
-	3350 5300 3750 5300
-Wire Wire Line
 	3350 5500 3750 5500
 Wire Wire Line
-	3350 5600 3750 5600
-Wire Wire Line
 	3350 5800 3750 5800
 Wire Wire Line
-	3350 5900 3750 5900
-Wire Wire Line
 	3350 6000 3750 6000
 Wire Wire Line
 	3350 6100 3750 6100
-Wire Wire Line
-	3350 6200 3750 6200
 Wire Wire Line
 	6000 2700 6000 2600
@@
 Wire Wire Line
 	5850 2700 6000 2700
+Text Label 5850 3600 0    50   ~ 0
+CAM1_D0-
+Text Label 5850 3800 0    50   ~ 0
+CAM1_D0+
+Wire Wire Line
+	5850 4000 6350 4000
+Wire Wire Line
+	5850 4300 6350 4300
+Wire Wire Line
+	5850 4400 6250 4400
+Wire Wire Line
+	5850 4200 6250 4200
+Wire Wire Line
+	5850 4100 6250 4100
+Wire Wire Line
+	5850 3900 6250 3900
+Wire Wire Line
+	5850 3800 6250 3800
+Wire Wire Line
+	5850 3700 6350 3700
+Wire Wire Line
+	5850 3600 6250 3600
+Wire Wire Line
+	5850 3500 6250 3500
+Text Label 5850 3900 0    50   ~ 0
+CAM1_D1-
+Text Label 5850 4100 0    50   ~ 0
+CAM1_D1+
+Text Label 5850 4200 0    50   ~ 0
+CAM1_C-
 Text Label 5850 4400 0    50   ~ 0
-CAM1_D0-
-Text Label 5850 4200 0    50   ~ 0
-CAM1_D0+
-Wire Wire Line
-	5850 4000 6350 4000
-Wire Wire Line
-	5850 4300 6350 4300
-Wire Wire Line
-	5850 4400 6250 4400
-Wire Wire Line
-	5850 4200 6250 4200
-Wire Wire Line
-	5850 4100 6250 4100
-Wire Wire Line
-	5850 3900 6250 3900
-Wire Wire Line
-	5850 3800 6250 3800
-Wire Wire Line
-	5850 3700 6350 3700
-Wire Wire Line
-	5850 3600 6250 3600
-Wire Wire Line
-	5850 3500 6250 3500
-Text Label 5850 4100 0    50   ~ 0
-CAM1_D1-
-Text Label 5850 3900 0    50   ~ 0
-CAM1_D1+
-Text Label 5850 3800 0    50   ~ 0
-CAM1_C-
-Text Label 5850 3600 0    50   ~ 0
 CAM1_C+
 Text Label 5850 3500 0    50   ~ 0
@@
 Wire Wire Line
 	5850 6550 6250 6550
+Text Label 5850 5750 0    50   ~ 0
+CAM2_D0-
+Text Label 5850 5950 0    50   ~ 0
+CAM2_D0+
+Text Label 5850 6050 0    50   ~ 0
+CAM2_D1-
+Text Label 5850 6250 0    50   ~ 0
+CAM2_D1+
+Text Label 5850 6350 0    50   ~ 0
+CAM2_C-
 Text Label 5850 6550 0    50   ~ 0
-CAM2_D0-
-Text Label 5850 6350 0    50   ~ 0
-CAM2_D0+
-Text Label 5850 6250 0    50   ~ 0
-CAM2_D1-
-Text Label 5850 6050 0    50   ~ 0
-CAM2_D1+
-Text Label 5850 5950 0    50   ~ 0
-CAM2_C-
-Text Label 5850 5750 0    50   ~ 0
 CAM2_C+
 Text Label 5850 5650 0    50   ~ 0
@@
 Powering the servos with the Pis +5V
 Text Notes 6600 6200 0    50   ~ 0
-Trying to match sensitive signals\nwith shielded twisted pairs
+Trying to match differential signals\nwith shielded twisted pairs
 Text Notes 8200 4500 0    50   ~ 0
 If need be, we can solder to \nthe top Pi's GPIOs as a last ditch fix for something\n
@@
 Text Notes 8130 7635 0    39   Italic 8
 Oct. 2018
+Wire Wire Line
+	3750 3550 3350 3550
+Wire Wire Line
+	3750 3250 3350 3250
+Wire Wire Line
+	3750 2950 3350 2950
+Wire Wire Line
+	3750 2650 3350 2650
+Wire Wire Line
+	3250 4150 3750 4150
+Connection ~ 3250 4150
+Wire Wire Line
+	3250 4150 3250 4250
+Wire Wire Line
+	3250 4250 3750 4250
+Connection ~ 3250 4250
+Wire Wire Line
+	3250 3150 3750 3150
+Wire Wire Line
+	3250 3150 3250 3450
+Wire Wire Line
+	3250 3450 3750 3450
+Connection ~ 3250 3450
+Wire Wire Line
+	3250 3450 3250 3750
+Wire Wire Line
+	3250 3750 3750 3750
+Connection ~ 3250 3750
+Wire Wire Line
+	3250 3750 3250 4050
+Wire Wire Line
+	3250 4050 3750 4050
+Connection ~ 3250 4050
+Wire Wire Line
+	3250 4050 3250 4150
+Wire Wire Line
+	3250 4250 3250 5300
+Wire Wire Line
+	3750 5700 3350 5700
+Wire Wire Line
+	3750 5400 3350 5400
+Wire Wire Line
+	3750 5100 3350 5100
+Wire Wire Line
+	3750 4800 3350 4800
+Wire Wire Line
+	3250 5300 3750 5300
+Connection ~ 3250 5300
+Wire Wire Line
+	3250 5900 3750 5900
+Connection ~ 3250 5900
+Wire Wire Line
+	3250 5900 3250 6200
+Wire Wire Line
+	3250 6200 3750 6200
+Connection ~ 3250 6200
+Wire Wire Line
+	3250 6200 3250 6300
+Wire Wire Line
+	3250 5600 3750 5600
+Wire Wire Line
+	3250 5300 3250 5600
+Connection ~ 3250 5600
+Wire Wire Line
+	3250 5600 3250 5900
 $EndSCHEMATC

Commit message: DC-DC Board Final
99% Done the first DC-DC Board. Just need to double check everything!!
Other:
- note removed: "Eastern Edge Robotics"

Commit message: Started DC-DC with Micro
Picked out microcontroller maybe? Still gotta decide if I want to use the 5x5 vs the 7x7.
Parts:
- J1, J2: footprint EER:MOLEX_0705530001 -> EER:70553-02
Changed lines of the file:
@@
 F 1 "Camera FPC Connector" H 3950 3050 50  0000 C CNN
 F 2 "EER:CON15_1X15_DRB_SFW" H 3750 4800 50  0001 C CNN
-F 3 "" H 3750 4800 50  0001 C CNN
+F 3 "609-1905-1-ND" H 3750 4800 50  0001 C CNN
 	1    3750 4800
 	1    0    0    -1
@@
 F 0 "J2" H 3600 1600 50  0000 C CNN
 F 1 "Servo Input" H 3600 1700 50  0000 C CNN
-F 2 "EER:MOLEX_0705530001" H 3600 1950 50  0001 C CNN
+F 2 "EER:70553-02" H 3600 1950 50  0001 C CNN
 F 3 "WM4900-ND" H 3600 1950 50  0001 C CNN
 	1    3600 1950
@@
 F 0 "J1" H 3600 1100 50  0000 C CNN
 F 1 "Servo Input" H 3600 1200 50  0000 C CNN
-F 2 "EER:MOLEX_0705530001" H 3600 1450 50  0001 C CNN
+F 2 "EER:70553-02" H 3600 1450 50  0001 C CNN
 F 3 "WM4900-ND" H 3600 1450 50  0001 C CNN
 	1    3600 1450
@@
 F 1 "Raspberry Pi GPIO" H 7400 3050 50  0000 C CNN
 F 2 "Pin_Headers:Pin_Header_Straight_2x20_Pitch2.54mm" H 7400 4250 50  0001 C CNN
-F 3 "~" H 7400 4250 50  0001 C CNN
+F 3 "S9200-ND" H 7400 4250 50  0001 C CNN
 	1    7400 4250
 	1    0    0    -1
