File: PCBs/DC-DC Board - Micro/DC-DC Board Micro.sch (KiCad schematic (older format))
At the start: 36 parts, among them J1 Conn_01x01, J2 Conn_01x01, J3 Conn_01x01, J4 Conn_01x01, J5 Conn_01x02, J6 Conn_01x02, Q1 Q_NMOS_GDS, U1 DBQ0135V2, U2 ACS711, U3 NCP551, U4 TLV733P

Commit message: Started DC-DC with Micro
Picked out microcontroller maybe? Still gotta decide if I want to use the 5x5 vs the 7x7.
Parts:
- removed C5, C7: 1uF, Capacitors_SMD:C_0805, symbol Device:C
- removed J6: Conn_01x02, EER:70553-02, symbol Connector_Generic:Conn_01x02
- removed TP1, TP2: TestPoint, Testpoints:TestPoint_Pad_D1.0mm, symbol Connector:TestPoint
- removed U3: NCP551, TO_SOT_Packages_SMD:SOT-23-5, symbol EER:MC33375
- added J6: Conn_01x03, EER:70553-03, symbol Connector_Generic:Conn_01x03
Connections:
- net labels added: +5V, VIOUT1, VIOUT2, VIOUT3
- net labels removed: 5V, VIOUT
- wire segments 148 -> 137
Other:
- note added: "5V-3V3 for Current Sensor and uC\n\n"
- note added: "Current Sensor Input\n"
- note added: "DC-DC Board - Micro\n"
- note added: "SAMD21 uC\n"
- note removed: "12V-5V-3V3 for Current Sensor\n"
- note removed: "Current Sensor Output\n"
- note removed: "DC-DC Board - No Micro\n"
- moved on the sheet: U4

Commit message: DC-DC Mirco Updates
Parts:
- C9: renamed from C11; value 1uF -> 10uF
- D1: value LED -> GRN
- D2: renamed from D3; value LED -> BLUE
- renumbered C12 to C10, C13 to C11, C9 to C5, C8 to C7, C10 to C8, J2 to J1, J1 to J2, J5 to J3, J6 to J4, J4 to J5, J3 to J6, R2 to R1, R1 to R2, R7 to R3, R8 to R4, R9 to R5, R3 to R6, R4 to R7, R6 to R8, U2 to U1, U1 to U2, U4 to U3
Connections:
- wire segments 137 -> 144
Other:
- moved on the sheet: U3

Commit message: DC-DC Boards 99%
Both boards are pretty much done. They just need a few double checks and some BOM work has to be done for the Micro Board.
Parts:
- C10, C11, C9: footprint Capacitors_SMD:C_0805 -> Capacitors_SMD:C_0603
Changed lines of the file:
@@
 F 0 "C9" H 9065 5646 50  0000 L CNN
 F 1 "10uF" H 9065 5555 50  0000 L CNN
-F 2 "Capacitors_SMD:C_0805" H 8988 5450 50  0001 C CNN
+F 2 "Capacitors_SMD:C_0603" H 8988 5450 50  0001 C CNN
 F 3 "490-10748-1-ND" H 8950 5600 50  0001 C CNN
 	1    8950 5600
@@
 F 0 "C10" H 9465 5646 50  0000 L CNN
 F 1 "1uF" H 9465 5555 50  0000 L CNN
-F 2 "Capacitors_SMD:C_0805" H 9388 5450 50  0001 C CNN
+F 2 "Capacitors_SMD:C_0603" H 9388 5450 50  0001 C CNN
 F 3 "399-1284-1-ND" H 9350 5600 50  0001 C CNN
 	1    9350 5600
@@
 F 0 "C11" H 9915 5646 50  0000 L CNN
 F 1 "0.1uF" H 9915 5555 50  0000 L CNN
-F 2 "Capacitors_SMD:C_0805" H 9838 5450 50  0001 C CNN
+F 2 "Capacitors_SMD:C_0603" H 9838 5450 50  0001 C CNN
 F 3 "399-1169-1-ND" H 9800 5600 50  0001 C CNN
 	1    9800 5600
