File: PCBs/DC-DC Board - Micro/SAMD21.sch (KiCad schematic (older format))
At the start: 2 parts, among them J7 USB_B_Mini, U3 ATSAMD21G16B-MFT

Commit message: DC-DC Mirco Updates
Parts:
- removed U3: ATSAMD21G16B-MFT, Digikey:QFN-48-1EP_7x7mm, symbol EER:ATSAMD21G16B-MFT
- added C12, C14: 10uF, Capacitors_SMD:C_0805, symbol Device:C
- added C13, C21: 0.1uF, Capacitors_SMD:C_0805, symbol Device:C
- added C15, C16, C17, C20: 1uF, Capacitors_SMD:C_0805, symbol Device:C
- added C18, C19: 22pF, Capacitors_SMD:C_0603, symbol Device:C
- added D3: RED, LEDs:LED_0805, symbol Device:LED
- added D4: ORNGE, LEDs:LED_0805, symbol Device:LED
- added F1: 500mA, Fuse_Holders_and_Fuses:Fuse_SMD1206_Reflow, symbol Device:Fuse
- added J8: Conn_02x05_Odd_Even, Pin_Headers:Pin_Header_Straight_2x05_Pitch1.27mm, symbol Connector_Generic:Conn_02x05_Odd_Even
- added L1, L2: Ferrite_Bead, Inductors_SMD:L_0805, symbol Device:Ferrite_Bead
- added R10: 10k, Resistors_SMD:R_0805, symbol Device:R_US
- added R11, R9: 330, Resistors_SMD:R_0805, symbol Device:R_US
- added SW1: SW_Push, Buttons_Switches_SMD:SW_SPST_EVQP0, symbol Switch:SW_Push
- added U4: ATSAMD21E16L-MFT, Digikey:QFN-32-1EP_5x5mm, symbol EER:ATSAMD21E16L-MFT
- added Y1: 32.7680kHz, Crystals:Crystal_SMD_3215-2pin_3.2x1.5mm, symbol Device:Crystal
- J7: footprint Digikey:USB_Mini_B_Female_UJ2-MBH-1-SMT-TR -> EER:32005-201
Connections:
- net labels added: +3.3V, +5V, 3V3_FILT, GND, SCL, SDA, SWCLK, SWDIO, USB+, USB-, VIOUT1, VIOUT2, VIOUT3, ~RESET~
- wire segments 0 -> 100
- no-connect marks 0 -> 19
Other:
- note added: "AIN Filtering\n\n"
- note added: "AIN5"
- note added: "AIN6"
- note added: "AIN7"
- note added: "PWR Filtering\n\n"
- note added: "Pinout for the SAMD21E"
- note added: "SWD Interface\n"
- note added: "TESTIO"
- note added: "USB PWR"
- moved on the sheet: J7

Commit message: DC-DC Boards 99%
Both boards are pretty much done. They just need a few double checks and some BOM work has to be done for the Micro Board.
Parts:
- C12, C13, C14, C15, C16, C17, C20, C21: footprint Capacitors_SMD:C_0805 -> Capacitors_SMD:C_0603
- R11, R9: footprint Resistors_SMD:R_0805 -> Capacitors_SMD:C_0603
- SW1: footprint Buttons_Switches_SMD:SW_SPST_EVQP0 -> Buttons_Switches_SMD:SW_SPST_EVQPE1
Changed lines of the file:
@@
 F 1 "USB_B_Mini" H 1555 3076 50  0000 C CNN
 F 2 "EER:32005-201" H 1650 2650 50  0001 C CNN
-F 3 "~" H 1650 2650 50  0001 C CNN
+F 3 "151-1206-1-ND" H 1650 2650 50  0001 C CNN
 	1    1500 2700
 	1    0    0    -1
@@
 F 0 "C12" H 2365 1496 50  0000 L CNN
 F 1 "10uF" H 2365 1405 50  0000 L CNN
-F 2 "Capacitors_SMD:C_0805" H 2288 1300 50  0001 C CNN
+F 2 "Capacitors_SMD:C_0603" H 2288 1300 50  0001 C CNN
 F 3 "490-10748-1-ND" H 2250 1450 50  0001 C CNN
 	1    2250 1450
@@
 F 0 "C13" H 2815 1496 50  0000 L CNN
 F 1 "0.1uF" H 2815 1405 50  0000 L CNN
-F 2 "Capacitors_SMD:C_0805" H 2738 1300 50  0001 C CNN
+F 2 "Capacitors_SMD:C_0603" H 2738 1300 50  0001 C CNN
 F 3 "399-1169-1-ND" H 2700 1450 50  0001 C CNN
 	1    2700 1450
@@
 F 0 "SW1" V 5146 4552 50  0000 R CNN
 F 1 "SW_Push" V 5055 4552 50  0000 R CNN
-F 2 "Buttons_Switches_SMD:SW_SPST_EVQP0" H 5100 4800 50  0001 C CNN
-F 3 "" H 5100 4800 50  0001 C CNN
+F 2 "Buttons_Switches_SMD:SW_SPST_EVQPE1" H 5100 4800 50  0001 C CNN
+F 3 "401-1707-1-ND" H 5100 4800 50  0001 C CNN
 	1    5100 4600
 	0    -1   -1   0
@@
 F 1 "500mA" V 2056 2500 50  0000 C CNN
 F 2 "Fuse_Holders_and_Fuses:Fuse_SMD1206_Reflow" V 1880 2500 50  0001 C CNN
-F 3 "~" H 1950 2500 50  0001 C CNN
+F 3 "507-1075-1-ND" H 1950 2500 50  0001 C CNN
 	1    1950 2500
 	0    -1   -1   0
@@
 F 0 "C14" H 2915 2896 50  0000 L CNN
 F 1 "10uF" H 2915 2805 50  0000 L CNN
-F 2 "Capacitors_SMD:C_0805" H 2838 2700 50  0001 C CNN
+F 2 "Capacitors_SMD:C_0603" H 2838 2700 50  0001 C CNN
 F 3 "490-10748-1-ND" H 2800 2850 50  0001 C CNN
 	1    2800 2850
@@
 F 0 "C15" H 3365 2896 50  0000 L CNN
 F 1 "1uF" H 3365 2805 50  0000 L CNN
-F 2 "Capacitors_SMD:C_0805" H 3288 2700 50  0001 C CNN
+F 2 "Capacitors_SMD:C_0603" H 3288 2700 50  0001 C CNN
 F 3 "399-1284-1-ND" H 3250 2850 50  0001 C CNN
 	1    3250 2850
@@
 F 0 "R9" H 3868 2896 50  0000 L CNN
 F 1 "330" H 3868 2805 50  0000 L CNN
-F 2 "Resistors_SMD:R_0805" V 3840 2840 50  0001 C CNN
+F 2 "Capacitors_SMD:C_0603" V 3840 2840 50  0001 C CNN
 F 3 "~" H 3800 2850 50  0001 C CNN
 	1    3800 2850
@@
 F 0 "C21" H 7415 1846 50  0000 L CNN
 F 1 "0.1uF" H 7415 1755 50  0000 L CNN
-F 2 "Capacitors_SMD:C_0805" H 7338 1650 50  0001 C CNN
+F 2 "Capacitors_SMD:C_0603" H 7338 1650 50  0001 C CNN
 F 3 "399-1169-1-ND" H 7300 1800 50  0001 C CNN
 	1    7300 1800
@@
 F 0 "R11" V 5395 3450 50  0000 C CNN
 F 1 "330" V 5486 3450 50  0000 C CNN
-F 2 "Resistors_SMD:R_0805" V 5640 3440 50  0001 C CNN
+F 2 "Capacitors_SMD:C_0603" V 5640 3440 50  0001 C CNN
 F 3 "~" H 5600 3450 50  0001 C CNN
 	1    5600 3450
@@
 F 0 "C16" H 4315 1446 50  0000 L CNN
 F 1 "1uF" H 4315 1355 50  0000 L CNN
-F 2 "Capacitors_SMD:C_0805" H 4238 1250 50  0001 C CNN
+F 2 "Capacitors_SMD:C_0603" H 4238 1250 50  0001 C CNN
 F 3 "399-1284-1-ND" H 4200 1400 50  0001 C CNN
 	1    4200 1400
@@
 F 0 "C17" H 4815 1446 50  0000 L CNN
 F 1 "1uF" H 4815 1355 50  0000 L CNN
-F 2 "Capacitors_SMD:C_0805" H 4738 1250 50  0001 C CNN
+F 2 "Capacitors_SMD:C_0603" H 4738 1250 50  0001 C CNN
 F 3 "399-1284-1-ND" H 4700 1400 50  0001 C CNN
 	1    4700 1400
@@
 F 0 "C20" H 5315 1446 50  0000 L CNN
 F 1 "1uF" H 5315 1355 50  0000 L CNN
-F 2 "Capacitors_SMD:C_0805" H 5238 1250 50  0001 C CNN
+F 2 "Capacitors_SMD:C_0603" H 5238 1250 50  0001 C CNN
 F 3 "399-1284-1-ND" H 5200 1400 50  0001 C CNN
 	1    5200 1400

Commit message: Finished Component Selection DC-DC - Micro
Parts:
- F1: footprint Fuse_Holders_and_Fuses:Fuse_SMD1206_Reflow -> EER:Fuse_SMD1206_Reflow
- R11: value 330 -> 150; footprint Capacitors_SMD:C_0603 -> Resistors_SMD:R_0603
- R9: footprint Capacitors_SMD:C_0603 -> Resistors_SMD:R_0603
- SW1: footprint Buttons_Switches_SMD:SW_SPST_EVQPE1 -> EER:SW_SPST_EVQPE1
- U4: footprint Digikey:QFN-32-1EP_5x5mm -> EER:QFN-32-1EP_5x5mm
- Y1: footprint Crystals:Crystal_SMD_3215-2pin_3.2x1.5mm -> EER:Crystal_SMD_3215-2pin_3.2x1.5mm
Changed lines of the file:
@@
 F 0 "U4" H 6400 2400 60  0000 C CNN
 F 1 "ATSAMD21E16L-MFT" H 7550 3050 60  0000 C CNN
-F 2 "Digikey:QFN-32-1EP_5x5mm" H 7900 3550 60  0001 L CNN
+F 2 "EER:QFN-32-1EP_5x5mm" H 7900 3550 60  0001 L CNN
 F 3 "1611-ATSAMD21E16L-MFTCT-ND" H 7900 3650 60  0001 L CNN
 F 4 "Active" H 6700 4650 60  0001 L CNN "Status"
@@
 F 1 "10uF" H 2365 1405 50  0000 L CNN
 F 2 "Capacitors_SMD:C_0603" H 2288 1300 50  0001 C CNN
-F 3 "490-10748-1-ND" H 2250 1450 50  0001 C CNN
+F 3 "490-7201-1-ND" H 2250 1450 50  0001 C CNN
 	1    2250 1450
 	1    0    0    -1
@@
 F 1 "0.1uF" H 2815 1405 50  0000 L CNN
 F 2 "Capacitors_SMD:C_0603" H 2738 1300 50  0001 C CNN
-F 3 "399-1169-1-ND" H 2700 1450 50  0001 C CNN
+F 3 "1276-1258-1-ND" H 2700 1450 50  0001 C CNN
 	1    2700 1450
 	1    0    0    -1
@@
 F 0 "SW1" V 5146 4552 50  0000 R CNN
 F 1 "SW_Push" V 5055 4552 50  0000 R CNN
-F 2 "Buttons_Switches_SMD:SW_SPST_EVQPE1" H 5100 4800 50  0001 C CNN
+F 2 "EER:SW_SPST_EVQPE1" H 5100 4800 50  0001 C CNN
 F 3 "401-1707-1-ND" H 5100 4800 50  0001 C CNN
 	1    5100 4600
@@
 F 0 "F1" V 2147 2500 50  0000 C CNN
 F 1 "500mA" V 2056 2500 50  0000 C CNN
-F 2 "Fuse_Holders_and_Fuses:Fuse_SMD1206_Reflow" V 1880 2500 50  0001 C CNN
+F 2 "EER:Fuse_SMD1206_Reflow" V 1880 2500 50  0001 C CNN
 F 3 "507-1075-1-ND" H 1950 2500 50  0001 C CNN
 	1    1950 2500
@@
 F 1 "10uF" H 2915 2805 50  0000 L CNN
 F 2 "Capacitors_SMD:C_0603" H 2838 2700 50  0001 C CNN
-F 3 "490-10748-1-ND" H 2800 2850 50  0001 C CNN
+F 3 "490-7201-1-ND" H 2800 2850 50  0001 C CNN
 	1    2800 2850
 	1    0    0    -1
@@
 F 1 "1uF" H 3365 2805 50  0000 L CNN
 F 2 "Capacitors_SMD:C_0603" H 3288 2700 50  0001 C CNN
-F 3 "399-1284-1-ND" H 3250 2850 50  0001 C CNN
+F 3 "1276-6524-1-ND" H 3250 2850 50  0001 C CNN
 	1    3250 2850
 	1    0    0    -1
@@
 F 0 "R9" H 3868 2896 50  0000 L CNN
 F 1 "330" H 3868 2805 50  0000 L CNN
-F 2 "Capacitors_SMD:C_0603" V 3840 2840 50  0001 C CNN
-F 3 "~" H 3800 2850 50  0001 C CNN
+F 2 "Resistors_SMD:R_0603" V 3840 2840 50  0001 C CNN
+F 3 "RHM330DCT-ND" H 3800 2850 50  0001 C CNN
 	1    3800 2850
 	1    0    0    -1
@@
 F 1 "RED" V 3747 3182 50  0000 R CNN
 F 2 "LEDs:LED_0805" H 3800 3300 50  0001 C CNN
-F 3 "~" H 3800 3300 50  0001 C CNN
+F 3 "732-4984-1-ND" H 3800 3300 50  0001 C CNN
 	1    3800 3300
 	0    -1   -1   0
@@
 F 0 "Y1" V 5104 2531 50  0000 L CNN
 F 1 "32.7680kHz" V 5195 2531 50  0000 L CNN
-F 2 "Crystals:Crystal_SMD_3215-2pin_3.2x1.5mm" H 5150 2400 50  0001 C CNN
+F 2 "EER:Crystal_SMD_3215-2pin_3.2x1.5mm" H 5150 2400 50  0001 C CNN
 F 3 "887-2605-1-ND" H 5150 2400 50  0001 C CNN
 	1    5150 2400
@@
 F 1 "22pF" V 4739 2200 50  0000 C CNN
 F 2 "Capacitors_SMD:C_0603" H 4938 2050 50  0001 C CNN
-F 3 "~" H 4900 2200 50  0001 C CNN
+F 3 "311-3925-1-ND" H 4900 2200 50  0001 C CNN
 	1    4900 2200
 	0    1    1    0
@@
 F 1 "22pF" V 4739 2600 50  0000 C CNN
 F 2 "Capacitors_SMD:C_0603" H 4938 2450 50  0001 C CNN
-F 3 "~" H 4900 2600 50  0001 C CNN
+F 3 "311-3925-1-ND" H 4900 2600 50  0001 C CNN
 	1    4900 2600
 	0    1    1    0
@@
 F 1 "0.1uF" H 7415 1755 50  0000 L CNN
 F 2 "Capacitors_SMD:C_0603" H 7338 1650 50  0001 C CNN
-F 3 "399-1169-1-ND" H 7300 1800 50  0001 C CNN
+F 3 "1276-1258-1-ND" H 7300 1800 50  0001 C CNN
 	1    7300 1800
 	1    0    0    -1
@@
 P 5600 3450
 F 0 "R11" V 5395 3450 50  0000 C CNN
-F 1 "330" V 5486 3450 50  0000 C CNN
-F 2 "Capacitors_SMD:C_0603" V 5640 3440 50  0001 C CNN
-F 3 "~" H 5600 3450 50  0001 C CNN
+F 1 "150" V 5486 3450 50  0000 C CNN
+F 2 "Resistors_SMD:R_0603" V 5640 3440 50  0001 C CNN
+F 3 "RHM150DCT-ND" H 5600 3450 50  0001 C CNN
 	1    5600 3450
 	0    1    1    0
@@
 F 1 "ORNGE" V 4897 3083 50  0000 R CNN
 F 2 "LEDs:LED_0805" H 4950 3200 50  0001 C CNN
-F 3 "~" H 4950 3200 50  0001 C CNN
+F 3 "160-1413-1-ND" H 4950 3200 50  0001 C CNN
 	1    4950 3200
 	0    -1   -1   0
@@
 F 1 "1uF" H 4315 1355 50  0000 L CNN
 F 2 "Capacitors_SMD:C_0603" H 4238 1250 50  0001 C CNN
-F 3 "399-1284-1-ND" H 4200 1400 50  0001 C CNN
+F 3 "1276-6524-1-ND" H 4200 1400 50  0001 C CNN
 	1    4200 1400
 	1    0    0    -1
@@
 F 1 "1uF" H 4815 1355 50  0000 L CNN
 F 2 "Capacitors_SMD:C_0603" H 4738 1250 50  0001 C CNN
-F 3 "399-1284-1-ND" H 4700 1400 50  0001 C CNN
+F 3 "1276-6524-1-ND" H 4700 1400 50  0001 C CNN
 	1    4700 1400
 	1    0    0    -1
@@
 F 1 "1uF" H 5315 1355 50  0000 L CNN
 F 2 "Capacitors_SMD:C_0603" H 5238 1250 50  0001 C CNN
-F 3 "399-1284-1-ND" H 5200 1400 50  0001 C CNN
+F 3 "1276-6524-1-ND" H 5200 1400 50  0001 C CNN
 	1    5200 1400
 	1    0    0    -1

Commit message: DC-DC Micro Touchups
Cleaned up layout and fixed orange test LED current limiting resistor.
Parts:
- R11: value 150 -> 680
Changed lines of the file:
@@
 P 5600 3450
 F 0 "R11" V 5395 3450 50  0000 C CNN
-F 1 "150" V 5486 3450 50  0000 C CNN
+F 1 "680" V 5486 3450 50  0000 C CNN
 F 2 "Resistors_SMD:R_0603" V 5640 3440 50  0001 C CNN
-F 3 "RHM150DCT-ND" H 5600 3450 50  0001 C CNN
+F 3 "RHM680DCT-ND" H 5600 3450 50  0001 C CNN
 	1    5600 3450
 	0    1    1    0

Commit message: Updated Mirco Stuff
Dodged a bullet
Parts:
- U4: value ATSAMD21E16L-MFT -> ATSAMD21E18A-MFTCT-ND; symbol EER:ATSAMD21E16L-MFT -> EER:ATSAMD21E18A-MFT
Changed lines of the file:
@@
 $EndComp
 $Comp
-L EER:ATSAMD21E16L-MFT U4
+L EER:ATSAMD21E18A-MFT U4
 U 1 1 5BCD2DFE
 P 6500 3450
 F 0 "U4" H 6400 2400 60  0000 C CNN
-F 1 "ATSAMD21E16L-MFT" H 7550 3050 60  0000 C CNN
+F 1 "ATSAMD21E18A-MFTCT-ND" H 7550 3050 60  0000 C CNN
 F 2 "EER:QFN-32-1EP_5x5mm" H 7900 3550 60  0001 L CNN
-F 3 "1611-ATSAMD21E16L-MFTCT-ND" H 7900 3650 60  0001 L CNN
+F 3 "ATSAMD21E18A-MFTCT-ND" H 7900 3650 60  0001 L CNN
 F 4 "Active" H 6700 4650 60  0001 L CNN "Status"
 	1    6500 3450
