File: PCBs/Maestro Adapter/Maestro Adapter.sch (KiCad schematic (older format))
At the start: 21 parts, among them J0 Conn_01x02_Female, J1 Conn_01x02_Female, J10 Conn_01x02_Female, J11 Conn_01x02_Female, J12 Conn_01x02_Female, J13 Conn_01x02_Female, J14 Conn_01x02_Female, J15 Conn_01x02_Female, J16 Conn_01x02_Female, J17 Conn_01x02_Female, J18 Conn_02x19_Counter_Clockwise, J2 Conn_01x02_Female, J3 Conn_01x02_Female, J4 Conn_01x02_Female, J5 Conn_01x02_Female, J6 Conn_01x02_Female, J7 Conn_01x02_Female, J8 Conn_01x02_Female, J9 Conn_01x02_Female

Commit message: Finalized the board
Parts:
- D1: footprint LED_SMD:LED_0805_2012Metric -> LEDs:LED_0805
- R1: footprint Resistor_SMD:R_0201_0603Metric -> Resistors_SMD:R_0603
Other:
- moved on the sheet: D1
Changed lines of the file:
@@
 L power:+5V #PWR0120
 U 1 1 5BD48154
-P 2600 3900
-F 0 "#PWR0120" H 2600 3750 50  0001 C CNN
-F 1 "+5V" V 2615 4028 50  0000 L CNN
-F 2 "" H 2600 3900 50  0001 C CNN
-F 3 "" H 2600 3900 50  0001 C CNN
-	1    2600 3900
+P 2650 3900
+F 0 "#PWR0120" H 2650 3750 50  0001 C CNN
+F 1 "+5V" V 2665 4028 50  0000 L CNN
+F 2 "" H 2650 3900 50  0001 C CNN
+F 3 "" H 2650 3900 50  0001 C CNN
+	1    2650 3900
 	0    1    1    0
 $EndComp
@@
 F 0 "R1" H 1320 1196 50  0000 L CNN
 F 1 "R" H 1320 1105 50  0000 L CNN
-F 2 "Resistor_SMD:R_0201_0603Metric" V 1180 1150 50  0001 C CNN
+F 2 "Resistors_SMD:R_0603" V 1180 1150 50  0001 C CNN
 F 3 "~" H 1250 1150 50  0001 C CNN
 	1    1250 1150
@@
 L Device:LED D1
 U 1 1 5BD48430
-P 1250 1450
-F 0 "D1" V 1288 1333 50  0000 R CNN
-F 1 "LED" V 1197 1333 50  0000 R CNN
-F 2 "LED_SMD:LED_0805_2012Metric" H 1250 1450 50  0001 C CNN
-F 3 "~" H 1250 1450 50  0001 C CNN
-	1    1250 1450
+P 1250 1550
+F 0 "D1" V 1288 1433 50  0000 R CNN
+F 1 "LED" V 1197 1433 50  0000 R CNN
+F 2 "LEDs:LED_0805" H 1250 1550 50  0001 C CNN
+F 3 "~" H 1250 1550 50  0001 C CNN
+	1    1250 1550
 	0    -1   -1   0
 $EndComp
@@
 L power:+5V #PWR0121
 U 1 1 5BD484FA
-P 1250 1000
-F 0 "#PWR0121" H 1250 850 50  0001 C CNN
-F 1 "+5V" H 1265 1173 50  0000 C CNN
-F 2 "" H 1250 1000 50  0001 C CNN
-F 3 "" H 1250 1000 50  0001 C CNN
-	1    1250 1000
+P 1250 900
+F 0 "#PWR0121" H 1250 750 50  0001 C CNN
+F 1 "+5V" H 1265 1073 50  0000 C CNN
+F 2 "" H 1250 900 50  0001 C CNN
+F 3 "" H 1250 900 50  0001 C CNN
+	1    1250 900
 	1    0    0    -1
 $EndComp
@@
 L power:GND #PWR0122
 U 1 1 5BD48554
-P 1250 1600
-F 0 "#PWR0122" H 1250 1350 50  0001 C CNN
-F 1 "GND" H 1255 1427 50  0000 C CNN
-F 2 "" H 1250 1600 50  0001 C CNN
-F 3 "" H 1250 1600 50  0001 C CNN
-	1    1250 1600
+P 1250 1800
+F 0 "#PWR0122" H 1250 1550 50  0001 C CNN
+F 1 "GND" H 1255 1627 50  0000 C CNN
+F 2 "" H 1250 1800 50  0001 C CNN
+F 3 "" H 1250 1800 50  0001 C CNN
+	1    1250 1800
 	1    0    0    -1
 $EndComp
+Wire Wire Line
+	2650 3900 2600 3900
+Wire Wire Line
+	1250 900  1250 1000
+Wire Wire Line
+	1250 1300 1250 1400
+Wire Wire Line
+	1250 1700 1250 1800
 $EndSCHEMATC
