File: PCBs/Maestro Adapter/Maestro Adapter.kicad_pcb (KiCad board)
At the start: 2 copper layers, 44.9 x 45.8 mm, 28 parts

Commit message: Gerbers and Maestro Fix
Added Gerbers for the maestro and fixed up the silkscreen.
Other:
- board text added: "18 Channel Maestro"
Changed lines of the file:
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@@
   (general
     (thickness 1.6)
-    (drawings 15)
+    (drawings 16)
     (tracks 123)
     (zones 0)
@@
   )
   (layers
-    (0 F.Cu signal hide)
-    (31 B.Cu signal hide)
-    (32 B.Adhes user hide)
-    (33 F.Adhes user hide)
-    (34 B.Paste user hide)
+    (0 F.Cu signal)
+    (31 B.Cu signal)
+    (32 B.Adhes user)
+    (33 F.Adhes user)
+    (34 B.Paste user)
     (35 F.Paste user hide)
-    (36 B.SilkS user hide)
+    (36 B.SilkS user)
     (37 F.SilkS user hide)
     (38 B.Mask user hide)
@@
     (visible_elements 7FFFF7FF)
     (pcbplotparams
-      (layerselection 0x010fc_ffffffff)
-      (usegerberextensions false)
+      (layerselection 0x010f0_ffffffff)
+      (usegerberextensions true)
       (usegerberattributes false)
       (usegerberadvancedattributes false)
@@
       (outputformat 1)
       (mirror false)
-      (drillshape 1)
+      (drillshape 0)
       (scaleselection 1)
-      (outputdirectory ""))
+      (outputdirectory "Gerbers/"))
   )
   (net 0 "")
@@
   (module EER:18ChannelMaestro (layer F.Cu)
     (at 80.19 168.22)
-    (fp_text reference "18 Channel Maestro" (at 9.4 -4.12) (layer B.SilkS)
-      (effects (font (size 1 1) (thickness 0.15)))
+    (fp_text reference "18 Channel Maestro" (at 9.4 -4.12) (layer B.SilkS) hide
+      (effects (font (size 1 1) (thickness 0.15)) (justify mirror))
     )
     (fp_text value "" (at 14.51 -49.71) (layer F.Fab)
@@
       (xy 1.277741 -0.528788) (xy 1.289465 -0.532567) (xy 1.293788 -0.532365)) (layer F.SilkS) (width 0.01))
   )
+  (gr_text "18 Channel Maestro" (at 94.3 164) (layer B.SilkS)
+    (effects (font (size 1.5 1.5) (thickness 0.3)) (justify mirror))
+  )
   (gr_text "Eastern Edge Robotics 2018/2019" (at 114.44 146.01 90) (layer B.SilkS)
