File: PCBs/Power Distribution Board/SAMD21PD.sch (KiCad schematic (older format))
At the start: 0 parts

Commit message: Schematic Finalized
99% done on the schematic, just needs to be checked over and touched-up.
Parts:
- added C? (x3): 10uF, symbol Device:C
- added C? (x13): 1uF, symbol Device:C
- added C? (x3): 0.1uF, symbol Device:C
- added C? (x2): 22pF, symbol Device:C
- added D?: RED, symbol Device:LED
- added D? (x2): ORNGE, symbol Device:LED
- added F?: 500mA, symbol Device:Fuse
- added J?: USB_B_Mini, symbol Connector:USB_B_Mini
- added J?: Conn_02x05_Odd_Even, symbol Connector_Generic:Conn_02x05_Odd_Even
- added L? (x2): Ferrite_Bead, symbol Device:Ferrite_Bead
- added R?: 330, symbol Device:R_US
- added R? (x2): 10k, symbol Device:R_US
- added R?: 680, symbol Device:R_US
- added SW?: SW_Push, symbol Switch:SW_Push
- added U?: ATSAMD21E16L-MFT, digikey-footprints:TQFP-48_7x7mm, symbol EER:ATSAMD21E16L-MFT
- added U?: TLV733P, Package_TO_SOT_SMD:SOT-23-5, symbol Regulator_Linear:TLV70018_SOT23-5
- added Y?: 32.7680kHz, symbol Device:Crystal
Connections:
- net labels added: +3V3, +5V, 3V3_FILT, GND, SWCLK, SWDIO, USB+, USB-, VIOUT1, VIOUT10, VIOUT2, VIOUT3, VIOUT4, VIOUT5, VIOUT6, VIOUT7, VIOUT8, VIOUT9, ~RESET
- wire segments 0 -> 162
- no-connect marks 0 -> 14
Other:
- note added: "AIN0\n"
- note added: "AIN1"
- note added: "AIN16\n"
- note added: "AIN17\n"
- note added: "AIN18\n"
- note added: "AIN19\n"
- note added: "AIN4"
- note added: "AIN5\n"
- note added: "AIN6\n"
- note added: "AIN7"
- note added: "Extra Filtering\n"
- note added: "PWR Indicator LEDs"
- note added: "Power Conversion"
- note added: "SAMD21E Pinout\n"
- note added: "SAMD21E uC\n\n"
- note added: "SWD Interface"
- note added: "TESTIO\n\n\n"
- note added: "USB Interface"
