File: PCBs/Power Distribution Board/SAMD21PD.sch (KiCad schematic (older format))
At the start: 37 parts, among them J28 USB_B_Mini, J29 Conn_02x05_Odd_Even, SW1 SW_Push, U11 TLV733P, U12 ATSAMD21E16L-MFT, Y1 32.7680kHz

Commit message: Initial Routing Finalized
Power Distribution Board is pretty much ready to go. Need to fix up the silkscreen and touch up routing but that will take only a little bit of time.
Changed lines of the file:
@@
 Text GLabel 5440 2860 0    50   Input ~ 0
 VIOUT1
+Text GLabel 5490 3760 0    50   Input ~ 0
+VIOUT2
 Text GLabel 5440 2960 0    50   Input ~ 0
-VIOUT2
+VIOUT3
+Text GLabel 5440 3660 0    50   Input ~ 0
+VIOUT4
 Text GLabel 5440 3060 0    50   Input ~ 0
-VIOUT3
+VIOUT5
+Text GLabel 5440 3560 0    50   Input ~ 0
+VIOUT6
 Text GLabel 5440 3160 0    50   Input ~ 0
-VIOUT4
+VIOUT7
+Text GLabel 5440 3460 0    50   Input ~ 0
+VIOUT8
 Text GLabel 5440 3260 0    50   Input ~ 0
-VIOUT5
+VIOUT9
 Text GLabel 5440 3360 0    50   Input ~ 0
-VIOUT6
-Text GLabel 5440 3460 0    50   Input ~ 0
-VIOUT7
-Text GLabel 5440 3560 0    50   Input ~ 0
-VIOUT8
-Text GLabel 5440 3660 0    50   Input ~ 0
-VIOUT9
-Text GLabel 5490 3760 0    50   Input ~ 0
 VIOUT10
 Wire Wire Line
@@
 Text Notes 4920 3300 0    50   ~ 0
 AIN6\n
-Text Notes 4920 3400 0    50   ~ 0
+Text Notes 4910 3400 0    50   ~ 0
 AIN7
 Text Notes 4900 3500 0    50   ~ 0
