File: PCBs/Power Distribution Board/SAMD21PD.sch (KiCad schematic (older format))
At the start: 37 parts, among them J28 USB_B_Mini, J29 Conn_02x05_Odd_Even, SW1 SW_Push, U11 TLV733P, U12 ATSAMD21E16L-MFT, Y1 32.7680kHz

Commit message: Updated Mirco Stuff
Dodged a bullet
Parts:
- U12: value ATSAMD21E16L-MFT -> ATSAMD21E18A-MFTCT-ND; symbol EER:ATSAMD21E16L-MFT -> EER:ATSAMD21E18A-MFT
Changed lines of the file:
@@
 SAMD21E uC\n\n
 $Comp
-L EER:ATSAMD21E16L-MFT U12
+L EER:ATSAMD21E18A-MFT U12
 U 1 1 5BD63CE2
 P 6420 3760
 F 0 "U12" H 6280 2680 60  0000 C CNN
-F 1 "ATSAMD21E16L-MFT" H 7490 3090 60  0000 C CNN
+F 1 "ATSAMD21E18A-MFTCT-ND" H 7490 3090 60  0000 C CNN
 F 2 "EER:QFN-32-1EP_5x5mm" H 7820 3860 60  0001 L CNN
-F 3 "1611-ATSAMD21E16L-MFTCT-ND" H 7820 3960 60  0001 L CNN
+F 3 "ATSAMD21E18A-MFTCT-ND" H 7820 3960 60  0001 L CNN
 F 4 "Active" H 6620 4960 60  0001 L CNN "Status"
 	1    6420 3760
